Commit message: m

File: diana_description/urdf/diana_soccer.xacro (robot description, xacro)
@@ -13,5 +13,5 @@
     <child link="pelvis"/>
    </joint>
-<!-- pelvis -->
+  <!-- pelvis -->
   <link name="pelvis">
    <collision>
@@ -72,5 +72,5 @@
     </inertial>
    </link>
-<joint name="waist_roll_joint" type="revolute">
+<joint name="waist_roll" type="revolute">
     <parent link="waist_fixed_link"/>
     <child link="waist_roll_link"/>
@@ -82,5 +82,5 @@
 <transmission name="tran0">
      <type>transmission_interface/SimpleTransmission</type>
-     <joint name="waist_roll_joint">
+     <joint name="waist_roll">
        <hardwareInterface>EffortJointInterface</hardwareInterface>
      </joint>
@@ -110,5 +110,5 @@
     </inertial>
    </link>
-<joint name="waist_yaw_joint" type="revolute">
+<joint name="waist_yaw" type="revolute">
     <parent link="waist_roll_link"/>
     <child link="waist_yaw_link"/>
@@ -120,5 +120,5 @@
 <transmission name="waist_yaw_tran">
      <type>transmission_interface/SimpleTransmission</type>
-     <joint name="waist_yaw_joint">
+     <joint name="waist_yaw">
        <hardwareInterface>EffortJointInterface</hardwareInterface>
      </joint>
@@ -149,5 +149,5 @@
    </link>
 <!-- head -->
-<joint name="head_yaw_joint" type="revolute">
+<joint name="head_yaw" type="revolute">
     <parent link="waist_yaw_link"/>
     <child link="head_yaw_link"/>
@@ -159,5 +159,5 @@
 <transmission name="head_yaw_tran">
      <type>transmission_interface/SimpleTransmission</type>
-     <joint name="head_yaw_joint">
+     <joint name="head_yaw">
        <hardwareInterface>EffortJointInterface</hardwareInterface>
      </joint>
@@ -187,5 +187,5 @@
     </inertial>
    </link>
-<joint name="head_pitch_joint" type="revolute">
+<joint name="head_pitch" type="revolute">
     <parent link="head_yaw_link"/>
     <child link="head_pitch_link"/>
@@ -197,5 +197,5 @@
 <transmission name="head_pitch_tran">
      <type>transmission_interface/SimpleTransmission</type>
-     <joint name="head_pitch_joint">
+     <joint name="head_pitch">
        <hardwareInterface>EffortJointInterface</hardwareInterface>
      </joint>
@@ -225,5 +225,5 @@
     </inertial>
    </link>
-<joint name="head_roll_joint" type="revolute">
+<joint name="head_roll" type="revolute">
     <parent link="head_pitch_link"/>
     <child link="head_roll_link"/>
@@ -235,5 +235,5 @@
 <transmission name="head_roll_tran">
      <type>transmission_interface/SimpleTransmission</type>
-     <joint name="head_roll_joint">
+     <joint name="head_roll">
        <hardwareInterface>EffortJointInterface</hardwareInterface>
      </joint>
@@ -264,5 +264,5 @@
    </link>
 <!-- left Arm -->
-<joint name="l_shoulder_pitch_joint" type="revolute">
+<joint name="l_shoulder_pitch" type="revolute">
     <parent link="waist_yaw_link"/>
     <child link="l_shoulder_pitch_link"/>
@@ -274,5 +274,5 @@
 <transmission name="l_shoulder_pitch_tran">
      <type>transmission_interface/SimpleTransmission</type>
-     <joint name="l_shoulder_pitch_joint">
+     <joint name="l_shoulder_pitch">
        <hardwareInterface>EffortJointInterface</hardwareInterface>
      </joint>
@@ -302,5 +302,5 @@
     </inertial>
    </link>
-<joint name="l_shoulder_roll_joint" type="revolute">
+<joint name="l_shoulder_roll" type="revolute">
     <parent link="l_shoulder_pitch_link"/>
     <child link="l_shoulder_roll_link"/>
@@ -312,5 +312,5 @@
 <transmission name="l_shoulder_roll_tran">
      <type>transmission_interface/SimpleTransmission</type>
-     <joint name="l_shoulder_roll_joint">
+     <joint name="l_shoulder_roll">
        <hardwareInterface>EffortJointInterface</hardwareInterface>
      </joint>
@@ -340,5 +340,5 @@
     </inertial>
   </link>
-<joint name="l_elbow_pitch_joint" type="revolute">
+<joint name="l_elbow_pitch" type="revolute">
     <parent link="l_shoulder_roll_link"/>
     <child link="l_elbow_pitch_link"/>
@@ -350,5 +350,5 @@
 <transmission name="l_elbow_pitch_tran">
      <type>transmission_interface/SimpleTransmission</type>
-     <joint name="l_elbow_pitch_joint">
+     <joint name="l_elbow_pitch">
        <hardwareInterface>EffortJointInterface</hardwareInterface>
      </joint>
@@ -379,5 +379,5 @@
   </link>
 <!-- right Arm -->
-<joint name="r_shoulder_pitch_joint" type="revolute">
+<joint name="r_shoulder_pitch" type="revolute">
     <parent link="waist_yaw_link"/>
     <child link="r_shoulder_pitch_link"/>
@@ -389,5 +389,5 @@
 <transmission name="r_shoulder_pitch_tran">
      <type>transmission_interface/SimpleTransmission</type>
-     <joint name="r_shoulder_pitch_joint">
+     <joint name="r_shoulder_pitch">
        <hardwareInterface>EffortJointInterface</hardwareInterface>
      </joint>
@@ -417,5 +417,5 @@
     </inertial>
    </link>
-<joint name="r_shoulder_roll_joint" type="revolute">
+<joint name="r_shoulder_roll" type="revolute">
     <parent link="r_shoulder_pitch_link"/>
     <child link="r_shoulder_roll_link"/>
@@ -427,5 +427,5 @@
 <transmission name="r_shoulder_roll_tran">
      <type>transmission_interface/SimpleTransmission</type>
-     <joint name="r_shoulder_roll_joint">
+     <joint name="r_shoulder_roll">
        <hardwareInterface>EffortJointInterface</hardwareInterface>
      </joint>
@@ -455,5 +455,5 @@
     </inertial>
   </link>
-<joint name="r_elbow_pitch_joint" type="revolute">
+<joint name="r_elbow_pitch" type="revolute">
     <parent link="r_shoulder_roll_link"/>
     <child link="r_elbow_pitch_link"/>
@@ -465,5 +465,5 @@
 <transmission name="r_elbow_pitch_tran">
      <type>transmission_interface/SimpleTransmission</type>
-     <joint name="r_elbow_pitch_joint">
+     <joint name="r_elbow_pitch">
        <hardwareInterface>EffortJointInterface</hardwareInterface>
      </joint>
@@ -494,5 +494,5 @@
   </link>
 <!-- left leg -->
-  <joint name="l_hip_pitch_joint" type="revolute">
+  <joint name="l_hip_pitch" type="revolute">
     <parent link="pelvis"/>
     <child link="l_hip_pitch_link"/>
@@ -504,5 +504,5 @@
   <transmission name="l_hip_pitch_tran">
      <type>transmission_interface/SimpleTransmission</type>
-     <joint name="l_hip_pitch_joint">
+     <joint name="l_hip_pitch">
        <hardwareInterface>EffortJointInterface</hardwareInterface>
      </joint>
@@ -532,5 +532,5 @@
     </inertial>
   </link>
-   <joint name="l_hip_roll_joint" type="revolute">
+   <joint name="l_hip_roll" type="revolute">
     <parent link="l_hip_pitch_link"/>
     <child link="l_hip_roll_link"/>
@@ -542,5 +542,5 @@
  <transmission name="l_hip_roll_tran">
      <type>transmission_interface/SimpleTransmission</type>
-     <joint name="l_hip_roll_joint">
+     <joint name="l_hip_roll">
        <hardwareInterface>EffortJointInterface</hardwareInterface>
      </joint>
@@ -570,5 +570,5 @@
     </inertial>
   </link>
-  <joint name="l_hip_yaw_joint" type="revolute">
+  <joint name="l_hip_yaw" type="revolute">
     <parent link="l_hip_roll_link"/>
     <child link="l_hip_yaw_link"/>
@@ -580,5 +580,5 @@
  <transmission name="l_hip_yaw_tran">
      <type>transmission_interface/SimpleTransmission</type>
-     <joint name="l_hip_yaw_joint">
+     <joint name="l_hip_yaw">
        <hardwareInterface>EffortJointInterface</hardwareInterface>
      </joint>
@@ -608,5 +608,5 @@
     </inertial>
   </link>
-  <joint name="l_knee_pitch_joint" type="revolute">
+  <joint name="l_knee_pitch" type="revolute">
     <parent link="l_hip_yaw_link"/>
     <child link="l_knee_pitch_link"/>
@@ -618,5 +618,5 @@
  <transmission name="l_knee_pitch_tran">
      <type>transmission_interface/SimpleTransmission</type>
-     <joint name="l_knee_pitch_joint">
+     <joint name="l_knee_pitch">
        <hardwareInterface>EffortJointInterface</hardwareInterface>
      </joint>
@@ -646,5 +646,5 @@
     </inertial>
   </link>
-  <joint name="l_ankle_pitch_joint" type="revolute">
+  <joint name="l_ankle_pitch" type="revolute">
     <parent link="l_knee_pitch_link"/>
     <child link="l_ankle_pitch_link"/>
@@ -656,5 +656,5 @@
  <transmission name="l_ankle_pitch_tran">
      <type>transmission_interface/SimpleTransmission</type>
-     <joint name="l_ankle_pitch_joint">
+     <joint name="l_ankle_pitch">
        <hardwareInterface>EffortJointInterface</hardwareInterface>
      </joint>
@@ -684,5 +684,5 @@
     </inertial>
   </link>
-  <joint name="l_ankle_roll_joint" type="revolute">
+  <joint name="l_ankle_roll" type="revolute">
     <parent link="l_ankle_pitch_link"/>
     <child link="l_ankle_roll_link"/>
@@ -694,5 +694,5 @@
  <transmission name="l_ankle_roll_tran">
      <type>transmission_interface/SimpleTransmission</type>
-     <joint name="l_ankle_roll_joint">
+     <joint name="l_ankle_roll">
        <hardwareInterface>EffortJointInterface</hardwareInterface>
      </joint>
@@ -748,5 +748,5 @@
   </link>
 <!-- right leg -->
-<joint name="r_hip_pitch_joint" type="revolute">
+<joint name="r_hip_pitch" type="revolute">
     <parent link="pelvis"/>
     <child link="r_hip_pitch_link"/>
@@ -758,5 +758,5 @@
    <transmission name="r_hip_pitch_tran">
      <type>transmission_interface/SimpleTransmission</type>
-     <joint name="r_hip_pitch_joint">
+     <joint name="r_hip_pitch">
        <hardwareInterface>EffortJointInterface</hardwareInterface>
      </joint>
@@ -787,5 +787,5 @@
 </link>
 <!-- - - - - - - - - - - - - - - - - - - - -->
-  <joint name="r_hip_roll_joint" type="revolute">
+  <joint name="r_hip_roll" type="revolute">
     <parent link="r_hip_pitch_link"/>
     <child link="r_hip_roll_link"/>
@@ -797,5 +797,5 @@
  <transmission name="r_hip_roll_tran">
      <type>transmission_interface/SimpleTransmission</type>
-     <joint name="r_hip_roll_joint">
+     <joint name="r_hip_roll">
        <hardwareInterface>EffortJointInterface</hardwareInterface>
      </joint>
@@ -826,5 +826,5 @@
   </link>
 <!-- - - - - - - - - - - - - - - - - - - - -->
-  <joint name="r_hip_yaw_joint" type="revolute">
+  <joint name="r_hip_yaw" type="revolute">
     <parent link="r_hip_roll_link"/>
     <child link="r_hip_yaw_link"/>
@@ -836,5 +836,5 @@
  <transmission name="r_hip_yaw_tran">
      <type>transmission_interface/SimpleTransmission</type>
-     <joint name="r_hip_yaw_joint">
+     <joint name="r_hip_yaw">
        <hardwareInterface>EffortJointInterface</hardwareInterface>
      </joint>
@@ -865,5 +865,5 @@
   </link>
 <!-- - - - - - - - - - - - - - - - - - - - -->
-  <joint name="r_knee_pitch_joint" type="revolute">
+  <joint name="r_knee_pitch" type="revolute">
     <parent link="r_hip_yaw_link"/>
     <child link="r_knee_pitch_link"/>
@@ -875,5 +875,5 @@
  <transmission name="r_knee_pitch_tran">
      <type>transmission_interface/SimpleTransmission</type>
-     <joint name="r_knee_pitch_joint">
+     <joint name="r_knee_pitch">
        <hardwareInterface>EffortJointInterface</hardwareInterface>
      </joint>
@@ -904,5 +904,5 @@
   </link>
 <!-- - - - - - - - - - - - - - - - - - - - -->
-  <joint name="r_ankle_pitch_joint" type="revolute">
+  <joint name="r_ankle_pitch" type="revolute">
     <parent link="r_knee_pitch_link"/>
     <child link="r_ankle_pitch_link"/>
@@ -914,5 +914,5 @@
  <transmission name="r_ankle_pitch_tran">
      <type>transmission_interface/SimpleTransmission</type>
-     <joint name="r_ankle_pitch_joint">
+     <joint name="r_ankle_pitch">
        <hardwareInterface>EffortJointInterface</hardwareInterface>
      </joint>
@@ -943,5 +943,5 @@
   </link>
 <!-- - - - - - - - - - - - - - - - - - - - -->
-  <joint name="r_ankle_roll_joint" type="revolute">
+  <joint name="r_ankle_roll" type="revolute">
     <parent link="r_ankle_pitch_link"/>
     <child link="r_ankle_roll_link"/>
@@ -953,5 +953,5 @@
    <transmission name="r_ankle_roll_tran">
      <type>transmission_interface/SimpleTransmission</type>
-     <joint name="r_ankle_roll_joint">
+     <joint name="r_ankle_roll">
        <hardwareInterface>EffortJointInterface</hardwareInterface>
      </joint>
