Commit message: m

File: diana_description/urdf/soccer_simulation.xacro (robot description, xacro)
@@ -6,12 +6,19 @@
   <xacro:include filename="$(find diana_description)/urdf/materials.xacro" />
   <!-- Used for fixing robot -->
-<link name = "base">
-</link>
-<joint name="world_fixed" type="fixed">
-    <origin xyz="0 0 0.65" rpy="0 0 0"/>
+  <link name="world">
+  </link>
+  <joint name="world_fixed" type="fixed">
+    <origin xyz="0 0 0" rpy="0 0 0"/>
+    <parent link="world"/>
+    <child link="base"/>
+  </joint>
+  <link name="base">
+  </link>
+  <joint name="base_fixed" type="fixed">
+    <origin xyz="0 0 0.723" rpy="0 0 0"/>
     <parent link="base"/>
     <child link="pelvis"/>
-   </joint>
-<!-- pelvis -->
+  </joint>
+  <!-- pelvis -->
   <link name="pelvis">
    <collision>
@@ -34,5 +41,5 @@
     </inertial>
   </link>
- <joint name="imu_fixed" type="fixed">
+  <joint name="imu_fixed" type="fixed">
     <parent link="pelvis"/>
     <child link="imu_link"/>
@@ -46,11 +53,11 @@
     </inertial>
   </link>
-<!-- chest -->
-<joint name="waist_fixed_joint" type="fixed">
+  <!-- chest -->
+  <joint name="waist_fixed" type="fixed">
     <parent link="pelvis"/>
     <child link="waist_fixed_link"/>
     <origin xyz="0 0 0" rpy="0 0 0"/>
-   </joint>
-<link name="waist_fixed_link">
+  </joint>
+  <link name="waist_fixed_link">
      <collision>
       <origin xyz="0 0 0" rpy="0 0 0"/>
@@ -71,6 +78,6 @@
       <inertia ixx="1.0" ixy="0.0" ixz="0.0" iyy="1.0" iyz="0.0" izz="1.0" />
     </inertial>
-   </link>
-<joint name="waist_roll_joint" type="revolute">
+  </link>
+  <joint name="waist_roll" type="revolute">
     <parent link="waist_fixed_link"/>
     <child link="waist_roll_link"/>
@@ -79,8 +86,8 @@
     <limit velocity="6.5" effort="1000" lower="${-pi/2}" upper="${pi}" />
     <dynamics damping = "0.7"/>
-   </joint>
-<transmission name="tran0">
-     <type>transmission_interface/SimpleTransmission</type>
-     <joint name="waist_roll_joint">
+  </joint>
+  <transmission name="tran0">
+     <type>transmission_interface/SimpleTransmission</type>
+     <joint name="waist_roll">
        <hardwareInterface>EffortJointInterface</hardwareInterface>
      </joint>
@@ -89,6 +96,6 @@
        <mechanicalReduction>1</mechanicalReduction>
      </actuator>
-   </transmission>
-<link name="waist_roll_link">
+  </transmission>
+  <link name="waist_roll_link">
    <collision>
       <origin xyz="0 0 0" rpy="0 0 0"/>
@@ -109,6 +116,6 @@
       <inertia ixx="1.0" ixy="0.0" ixz="0.0" iyy="1.0" iyz="0.0" izz="1.0" />
     </inertial>
-   </link>
-<joint name="waist_yaw_joint" type="revolute">
+  </link>
+  <joint name="waist_yaw" type="revolute">
     <parent link="waist_roll_link"/>
     <child link="waist_yaw_link"/>
@@ -118,7 +125,7 @@
     <dynamics damping = "0.7"/>
    </joint>
-<transmission name="waist_yaw_tran">
-     <type>transmission_interface/SimpleTransmission</type>
-     <joint name="waist_yaw_joint">
+  <transmission name="waist_yaw_tran">
+     <type>transmission_interface/SimpleTransmission</type>
+     <joint name="waist_yaw">
        <hardwareInterface>EffortJointInterface</hardwareInterface>
      </joint>
@@ -128,5 +135,5 @@
      </actuator>
    </transmission>
-<link name="waist_yaw_link">
+  <link name="waist_yaw_link">
    <collision>
       <origin xyz="0 0 0" rpy="0 0 0"/>
@@ -148,6 +155,6 @@
     </inertial>
    </link>
-<!-- head -->
-<joint name="head_yaw_joint" type="revolute">
+  <!-- head -->
+  <joint name="head_yaw" type="revolute">
     <parent link="waist_yaw_link"/>
     <child link="head_yaw_link"/>
@@ -157,7 +164,7 @@
     <dynamics damping = "0.7"/>
    </joint>
-<transmission name="head_yaw_tran">
-     <type>transmission_interface/SimpleTransmission</type>
-     <joint name="head_yaw_joint">
+  <transmission name="head_yaw_tran">
+     <type>transmission_interface/SimpleTransmission</type>
+     <joint name="head_yaw">
        <hardwareInterface>EffortJointInterface</hardwareInterface>
      </joint>
@@ -167,5 +174,5 @@
      </actuator>
    </transmission>
-<link name="head_yaw_link">
+  <link name="head_yaw_link">
    <collision>
       <origin xyz="0 0 0" rpy="0 0 0"/>
@@ -187,5 +194,5 @@
     </inertial>
    </link>
-<joint name="head_pitch_joint" type="revolute">
+  <joint name="head_pitch" type="revolute">
     <parent link="head_yaw_link"/>
     <child link="head_pitch_link"/>
@@ -195,7 +202,7 @@
     <dynamics damping = "0.7"/>
    </joint>
-<transmission name="head_pitch_tran">
-     <type>transmission_interface/SimpleTransmission</type>
-     <joint name="head_pitch_joint">
+  <transmission name="head_pitch_tran">
+     <type>transmission_interface/SimpleTransmission</type>
+     <joint name="head_pitch">
        <hardwareInterface>EffortJointInterface</hardwareInterface>
      </joint>
@@ -205,5 +212,5 @@
      </actuator>
    </transmission>
-<link name="head_pitch_link">
+  <link name="head_pitch_link">
    <collision>
       <origin xyz="0 0 0" rpy="0 0 0"/>
@@ -225,5 +232,5 @@
     </inertial>
    </link>
-<joint name="head_roll_joint" type="revolute">
+  <joint name="head_roll" type="revolute">
     <parent link="head_pitch_link"/>
     <child link="head_roll_link"/>
@@ -233,7 +240,7 @@
     <dynamics damping = "0.7"/>
    </joint>
-<transmission name="head_roll_tran">
-     <type>transmission_interface/SimpleTransmission</type>
-     <joint name="head_roll_joint">
+  <transmission name="head_roll_tran">
+     <type>transmission_interface/SimpleTransmission</type>
+     <joint name="head_roll">
        <hardwareInterface>EffortJointInterface</hardwareInterface>
      </joint>
@@ -243,5 +250,5 @@
      </actuator>
    </transmission>
-<link name="head_roll_link">
+  <link name="head_roll_link">
    <collision>
       <origin xyz="0 0 0" rpy="0 0 0"/>
@@ -263,6 +270,6 @@
     </inertial>
    </link>
-<!-- left Arm -->
-<joint name="l_shoulder_pitch_joint" type="revolute">
+  <!-- left Arm -->
+  <joint name="l_shoulder_pitch" type="revolute">
     <parent link="waist_yaw_link"/>
     <child link="l_shoulder_pitch_link"/>
@@ -274,5 +281,5 @@
 <transmission name="l_shoulder_pitch_tran">
      <type>transmission_interface/SimpleTransmission</type>
-     <joint name="l_shoulder_pitch_joint">
+     <joint name="l_shoulder_pitch">
        <hardwareInterface>EffortJointInterface</hardwareInterface>
      </joint>
@@ -302,5 +309,5 @@
     </inertial>
    </link>
-<joint name="l_shoulder_roll_joint" type="revolute">
+<joint name="l_shoulder_roll" type="revolute">
     <parent link="l_shoulder_pitch_link"/>
     <child link="l_shoulder_roll_link"/>
@@ -312,5 +319,5 @@
 <transmission name="l_shoulder_roll_tran">
      <type>transmission_interface/SimpleTransmission</type>
-     <joint name="l_shoulder_roll_joint">
+     <joint name="l_shoulder_roll">
        <hardwareInterface>EffortJointInterface</hardwareInterface>
      </joint>
@@ -340,5 +347,5 @@
     </inertial>
   </link>
-<joint name="l_elbow_pitch_joint" type="revolute">
+<joint name="l_elbow_pitch" type="revolute">
     <parent link="l_shoulder_roll_link"/>
     <child link="l_elbow_pitch_link"/>
@@ -350,5 +357,5 @@
 <transmission name="l_elbow_pitch_tran">
      <type>transmission_interface/SimpleTransmission</type>
-     <joint name="l_elbow_pitch_joint">
+     <joint name="l_elbow_pitch">
        <hardwareInterface>EffortJointInterface</hardwareInterface>
      </joint>
@@ -379,5 +386,5 @@
   </link>
 <!-- right Arm -->
-<joint name="r_shoulder_pitch_joint" type="revolute">
+<joint name="r_shoulder_pitch" type="revolute">
     <parent link="waist_yaw_link"/>
     <child link="r_shoulder_pitch_link"/>
@@ -389,5 +396,5 @@
 <transmission name="r_shoulder_pitch_tran">
      <type>transmission_interface/SimpleTransmission</type>
-     <joint name="r_shoulder_pitch_joint">
+     <joint name="r_shoulder_pitch">
        <hardwareInterface>EffortJointInterface</hardwareInterface>
      </joint>
@@ -417,5 +424,5 @@
     </inertial>
    </link>
-<joint name="r_shoulder_roll_joint" type="revolute">
+<joint name="r_shoulder_roll" type="revolute">
     <parent link="r_shoulder_pitch_link"/>
     <child link="r_shoulder_roll_link"/>
@@ -427,5 +434,5 @@
 <transmission name="r_shoulder_roll_tran">
      <type>transmission_interface/SimpleTransmission</type>
-     <joint name="r_shoulder_roll_joint">
+     <joint name="r_shoulder_roll">
        <hardwareInterface>EffortJointInterface</hardwareInterface>
      </joint>
@@ -455,5 +462,5 @@
     </inertial>
   </link>
-<joint name="r_elbow_pitch_joint" type="revolute">
+<joint name="r_elbow_pitch" type="revolute">
     <parent link="r_shoulder_roll_link"/>
     <child link="r_elbow_pitch_link"/>
@@ -465,5 +472,5 @@
 <transmission name="r_elbow_pitch_tran">
      <type>transmission_interface/SimpleTransmission</type>
-     <joint name="r_elbow_pitch_joint">
+     <joint name="r_elbow_pitch">
        <hardwareInterface>EffortJointInterface</hardwareInterface>
      </joint>
@@ -494,5 +501,5 @@
   </link>
 <!-- left leg -->
-  <joint name="l_hip_pitch_joint" type="revolute">
+  <joint name="l_hip_pitch" type="revolute">
     <parent link="pelvis"/>
     <child link="l_hip_pitch_link"/>
@@ -504,5 +511,5 @@
   <transmission name="l_hip_pitch_tran">
      <type>transmission_interface/SimpleTransmission</type>
-     <joint name="l_hip_pitch_joint">
+     <joint name="l_hip_pitch">
        <hardwareInterface>EffortJointInterface</hardwareInterface>
      </joint>
@@ -532,5 +539,5 @@
     </inertial>
   </link>
-   <joint name="l_hip_roll_joint" type="revolute">
+   <joint name="l_hip_roll" type="revolute">
     <parent link="l_hip_pitch_link"/>
     <child link="l_hip_roll_link"/>
@@ -542,5 +549,5 @@
  <transmission name="l_hip_roll_tran">
      <type>transmission_interface/SimpleTransmission</type>
-     <joint name="l_hip_roll_joint">
+     <joint name="l_hip_roll">
        <hardwareInterface>EffortJointInterface</hardwareInterface>
      </joint>
@@ -570,5 +577,5 @@
     </inertial>
   </link>
-  <joint name="l_hip_yaw_joint" type="revolute">
+  <joint name="l_hip_yaw" type="revolute">
     <parent link="l_hip_roll_link"/>
     <child link="l_hip_yaw_link"/>
@@ -580,5 +587,5 @@
  <transmission name="l_hip_yaw_tran">
      <type>transmission_interface/SimpleTransmission</type>
-     <joint name="l_hip_yaw_joint">
+     <joint name="l_hip_yaw">
        <hardwareInterface>EffortJointInterface</hardwareInterface>
      </joint>
@@ -608,5 +615,5 @@
     </inertial>
   </link>
-  <joint name="l_knee_pitch_joint" type="revolute">
+  <joint name="l_knee_pitch" type="revolute">
     <parent link="l_hip_yaw_link"/>
     <child link="l_knee_pitch_link"/>
@@ -618,5 +625,5 @@
  <transmission name="l_knee_pitch_tran">
      <type>transmission_interface/SimpleTransmission</type>
-     <joint name="l_knee_pitch_joint">
+     <joint name="l_knee_pitch">
        <hardwareInterface>EffortJointInterface</hardwareInterface>
      </joint>
@@ -646,5 +653,5 @@
     </inertial>
   </link>
-  <joint name="l_ankle_pitch_joint" type="revolute">
+  <joint name="l_ankle_pitch" type="revolute">
     <parent link="l_knee_pitch_link"/>
     <child link="l_ankle_pitch_link"/>
@@ -656,5 +663,5 @@
  <transmission name="l_ankle_pitch_tran">
      <type>transmission_interface/SimpleTransmission</type>
-     <joint name="l_ankle_pitch_joint">
+     <joint name="l_ankle_pitch">
        <hardwareInterface>EffortJointInterface</hardwareInterface>
      </joint>
@@ -684,5 +691,5 @@
     </inertial>
   </link>
-  <joint name="l_ankle_roll_joint" type="revolute">
+  <joint name="l_ankle_roll" type="revolute">
     <parent link="l_ankle_pitch_link"/>
     <child link="l_ankle_roll_link"/>
@@ -694,5 +701,5 @@
  <transmission name="l_ankle_roll_tran">
      <type>transmission_interface/SimpleTransmission</type>
-     <joint name="l_ankle_roll_joint">
+     <joint name="l_ankle_roll">
        <hardwareInterface>EffortJointInterface</hardwareInterface>
      </joint>
@@ -722,5 +729,5 @@
     </inertial>
   </link>
-  <joint name="l_last_joint" type="fixed">
+  <joint name="l_last" type="fixed">
     <parent link="l_ankle_roll_link"/>
     <child link="l_foot_link"/>
@@ -748,5 +755,5 @@
   </link>
 <!-- right leg -->
-<joint name="r_hip_pitch_joint" type="revolute">
+<joint name="r_hip_pitch" type="revolute">
     <parent link="pelvis"/>
     <child link="r_hip_pitch_link"/>
@@ -758,5 +765,5 @@
    <transmission name="r_hip_pitch_tran">
      <type>transmission_interface/SimpleTransmission</type>
-     <joint name="r_hip_pitch_joint">
+     <joint name="r_hip_pitch">
        <hardwareInterface>EffortJointInterface</hardwareInterface>
      </joint>
@@ -787,5 +794,5 @@
 </link>
 <!-- - - - - - - - - - - - - - - - - - - - -->
-  <joint name="r_hip_roll_joint" type="revolute">
+  <joint name="r_hip_roll" type="revolute">
     <parent link="r_hip_pitch_link"/>
     <child link="r_hip_roll_link"/>
@@ -797,5 +804,5 @@
  <transmission name="r_hip_roll_tran">
      <type>transmission_interface/SimpleTransmission</type>
-     <joint name="r_hip_roll_joint">
+     <joint name="r_hip_roll">
        <hardwareInterface>EffortJointInterface</hardwareInterface>
      </joint>
@@ -826,5 +833,5 @@
   </link>
 <!-- - - - - - - - - - - - - - - - - - - - -->
-  <joint name="r_hip_yaw_joint" type="revolute">
+  <joint name="r_hip_yaw" type="revolute">
     <parent link="r_hip_roll_link"/>
     <child link="r_hip_yaw_link"/>
@@ -836,5 +843,5 @@
  <transmission name="r_hip_yaw_tran">
      <type>transmission_interface/SimpleTransmission</type>
-     <joint name="r_hip_yaw_joint">
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