Commit message: organize joint_states and robot_states

File: diana_description/urdf/soccer_simulation.xacro (robot description, xacro)
@@ -22,5 +22,5 @@
   <!-- pelvis -->
   <link name="pelvis">
-   <collision>
+    <collision>
       <origin xyz="0 0 0" rpy="0 0 0"/>
       <geometry>
@@ -60,5 +60,5 @@
   </joint>
   <link name="waist_fixed_link">
-     <collision>
+    <collision>
       <origin xyz="0 0 0" rpy="0 0 0"/>
       <geometry>
@@ -87,5 +87,5 @@
     <dynamics damping = "0.7"/>
   </joint>
-  <transmission name="tran0">
+  <transmission name="waist_roll_tran">
      <type>transmission_interface/SimpleTransmission</type>
      <joint name="waist_roll">
@@ -98,5 +98,5 @@
   </transmission>
   <link name="waist_roll_link">
-   <collision>
+    <collision>
       <origin xyz="0 0 0" rpy="0 0 0"/>
       <geometry>
@@ -134,7 +134,7 @@
        <mechanicalReduction>1</mechanicalReduction>
      </actuator>
-   </transmission>
+  </transmission>
   <link name="waist_yaw_link">
-   <collision>
+    <collision>
       <origin xyz="0 0 0" rpy="0 0 0"/>
       <geometry>
@@ -154,5 +154,5 @@
       <inertia ixx="1.0" ixy="0.0" ixz="0.0" iyy="1.0" iyz="0.0" izz="1.0" />
     </inertial>
-   </link>
+  </link>
   <!-- head -->
   <joint name="head_yaw" type="revolute">
@@ -163,5 +163,5 @@
     <limit velocity="6.5" effort="1000" lower="${-pi/2}" upper="${pi/2}" />
     <dynamics damping = "0.7"/>
-   </joint>
+  </joint>
   <transmission name="head_yaw_tran">
      <type>transmission_interface/SimpleTransmission</type>
@@ -173,7 +173,7 @@
        <mechanicalReduction>1</mechanicalReduction>
      </actuator>
-   </transmission>
+  </transmission>
   <link name="head_yaw_link">
-   <collision>
+    <collision>
       <origin xyz="0 0 0" rpy="0 0 0"/>
       <geometry>
@@ -193,5 +193,5 @@
       <inertia ixx="1.0" ixy="0.0" ixz="0.0" iyy="1.0" iyz="0.0" izz="1.0" />
     </inertial>
-   </link>
+  </link>
   <joint name="head_pitch" type="revolute">
     <parent link="head_yaw_link"/>
@@ -201,5 +201,5 @@
     <limit velocity="6.5" effort="1000" lower="${-pi/2}" upper="${pi/2}" />
     <dynamics damping = "0.7"/>
-   </joint>
+  </joint>
   <transmission name="head_pitch_tran">
      <type>transmission_interface/SimpleTransmission</type>
@@ -213,5 +213,5 @@
    </transmission>
   <link name="head_pitch_link">
-   <collision>
+    <collision>
       <origin xyz="0 0 0" rpy="0 0 0"/>
       <geometry>
@@ -231,5 +231,5 @@
       <inertia ixx="1.0" ixy="0.0" ixz="0.0" iyy="1.0" iyz="0.0" izz="1.0" />
     </inertial>
-   </link>
+  </link>
   <joint name="head_roll" type="revolute">
     <parent link="head_pitch_link"/>
@@ -239,5 +239,5 @@
     <limit velocity="6.5" effort="1000" lower="${-pi/2}" upper="${pi/2}" />
     <dynamics damping = "0.7"/>
-   </joint>
+  </joint>
   <transmission name="head_roll_tran">
      <type>transmission_interface/SimpleTransmission</type>
@@ -249,7 +249,7 @@
        <mechanicalReduction>1</mechanicalReduction>
      </actuator>
-   </transmission>
+  </transmission>
   <link name="head_roll_link">
-   <collision>
+    <collision>
       <origin xyz="0 0 0" rpy="0 0 0"/>
       <geometry>
@@ -269,5 +269,5 @@
       <inertia ixx="1.0" ixy="0.0" ixz="0.0" iyy="1.0" iyz="0.0" izz="1.0" />
     </inertial>
-   </link>
+  </link>
   <!-- left Arm -->
   <joint name="l_shoulder_pitch" type="revolute">
@@ -278,6 +278,6 @@
     <limit velocity="6.5" effort="1000" lower="${-pi/2}" upper="${pi}" />
     <dynamics damping = "0.7"/>
-   </joint>
-<transmission name="l_shoulder_pitch_tran">
+  </joint>
+  <transmission name="l_shoulder_pitch_tran">
      <type>transmission_interface/SimpleTransmission</type>
      <joint name="l_shoulder_pitch">
@@ -288,7 +288,7 @@
        <mechanicalReduction>1</mechanicalReduction>
      </actuator>
-   </transmission>
-<link name="l_shoulder_pitch_link">
-   <collision>
+  </transmission>
+  <link name="l_shoulder_pitch_link">
+    <collision>
       <origin xyz="0 0 0" rpy="0 0 0"/>
       <geometry>
@@ -308,6 +308,6 @@
       <inertia ixx="1.0" ixy="0.0" ixz="0.0" iyy="1.0" iyz="0.0" izz="1.0" />
     </inertial>
-   </link>
-<joint name="l_shoulder_roll" type="revolute">
+  </link>
+  <joint name="l_shoulder_roll" type="revolute">
     <parent link="l_shoulder_pitch_link"/>
     <child link="l_shoulder_roll_link"/>
@@ -316,6 +316,6 @@
     <limit velocity="6.5" effort="1000" lower="${-pi/2}" upper="${pi}" />
     <dynamics damping = "0.7"/>
-   </joint>
-<transmission name="l_shoulder_roll_tran">
+  </joint>
+  <transmission name="l_shoulder_roll_tran">
      <type>transmission_interface/SimpleTransmission</type>
      <joint name="l_shoulder_roll">
@@ -326,7 +326,7 @@
        <mechanicalReduction>1</mechanicalReduction>
      </actuator>
-   </transmission>
-<link name="l_shoulder_roll_link">
-   <collision>
+  </transmission>
+  <link name="l_shoulder_roll_link">
+    <collision>
       <origin xyz="0 0 0" rpy="0 0 0"/>
       <geometry>
@@ -347,5 +347,5 @@
     </inertial>
   </link>
-<joint name="l_elbow_pitch" type="revolute">
+  <joint name="l_elbow_pitch" type="revolute">
     <parent link="l_shoulder_roll_link"/>
     <child link="l_elbow_pitch_link"/>
@@ -354,6 +354,6 @@
     <limit velocity="6.5" effort="1000" lower="${-pi/2}" upper="${pi/2}" />
     <dynamics damping = "0.7"/>
-   </joint>
-<transmission name="l_elbow_pitch_tran">
+  </joint>
+  <transmission name="l_elbow_pitch_tran">
      <type>transmission_interface/SimpleTransmission</type>
      <joint name="l_elbow_pitch">
@@ -364,7 +364,7 @@
        <mechanicalReduction>1</mechanicalReduction>
      </actuator>
-   </transmission>
-<link name="l_elbow_pitch_link">
-   <collision>
+  </transmission>
+  <link name="l_elbow_pitch_link">
+    <collision>
       <origin xyz="0 0 0" rpy="0 0 0"/>
       <geometry>
@@ -385,6 +385,6 @@
     </inertial>
   </link>
-<!-- right Arm -->
-<joint name="r_shoulder_pitch" type="revolute">
+  <!-- right Arm -->
+  <joint name="r_shoulder_pitch" type="revolute">
     <parent link="waist_yaw_link"/>
     <child link="r_shoulder_pitch_link"/>
@@ -393,6 +393,6 @@
     <limit velocity="6.5" effort="1000" lower="${-pi/2}" upper="${pi}" />
     <dynamics damping = "0.7"/>
-   </joint>
-<transmission name="r_shoulder_pitch_tran">
+  </joint>
+  <transmission name="r_shoulder_pitch_tran">
      <type>transmission_interface/SimpleTransmission</type>
      <joint name="r_shoulder_pitch">
@@ -403,7 +403,7 @@
        <mechanicalReduction>1</mechanicalReduction>
      </actuator>
-   </transmission>
-<link name="r_shoulder_pitch_link">
-   <collision>
+  </transmission>
+  <link name="r_shoulder_pitch_link">
+    <collision>
       <origin xyz="0 0 0" rpy="0 0 0"/>
       <geometry>
@@ -423,6 +423,6 @@
       <inertia ixx="1.0" ixy="0.0" ixz="0.0" iyy="1.0" iyz="0.0" izz="1.0" />
     </inertial>
-   </link>
-<joint name="r_shoulder_roll" type="revolute">
+  </link>
+  <joint name="r_shoulder_roll" type="revolute">
     <parent link="r_shoulder_pitch_link"/>
     <child link="r_shoulder_roll_link"/>
@@ -431,6 +431,6 @@
     <limit velocity="6.5" effort="1000" lower="${-pi/2}" upper="${pi}" />
     <dynamics damping = "0.7"/>
-   </joint>
-<transmission name="r_shoulder_roll_tran">
+  </joint>
+  <transmission name="r_shoulder_roll_tran">
      <type>transmission_interface/SimpleTransmission</type>
      <joint name="r_shoulder_roll">
@@ -441,7 +441,7 @@
        <mechanicalReduction>1</mechanicalReduction>
      </actuator>
-   </transmission>
-<link name="r_shoulder_roll_link">
-   <collision>
+  </transmission>
+  <link name="r_shoulder_roll_link">
+    <collision>
       <origin xyz="0 0 0" rpy="0 0 0"/>
       <geometry>
@@ -462,5 +462,5 @@
     </inertial>
   </link>
-<joint name="r_elbow_pitch" type="revolute">
+  <joint name="r_elbow_pitch" type="revolute">
     <parent link="r_shoulder_roll_link"/>
     <child link="r_elbow_pitch_link"/>
@@ -469,6 +469,6 @@
     <limit velocity="6.5" effort="1000" lower="${-pi/2}" upper="${pi/2}" />
     <dynamics damping = "0.7"/>
-   </joint>
-<transmission name="r_elbow_pitch_tran">
+  </joint>
+  <transmission name="r_elbow_pitch_tran">
      <type>transmission_interface/SimpleTransmission</type>
      <joint name="r_elbow_pitch">
@@ -479,7 +479,7 @@
        <mechanicalReduction>1</mechanicalReduction>
      </actuator>
-   </transmission>
-<link name="r_elbow_pitch_link">
-   <collision>
+  </transmission>
+  <link name="r_elbow_pitch_link">
+    <collision>
       <origin xyz="0 0 0" rpy="0 0 0"/>
       <geometry>
@@ -500,5 +500,5 @@
     </inertial>
   </link>
-<!-- left leg -->
+  <!-- left leg -->
   <joint name="l_hip_pitch" type="revolute">
     <parent link="pelvis"/>
@@ -508,5 +508,5 @@
     <limit velocity="6.5" effort="1000" lower="${-pi/2}" upper="${pi/2}" />
     <dynamics damping = "0.7"/>
-   </joint>
+  </joint>
   <transmission name="l_hip_pitch_tran">
      <type>transmission_interface/SimpleTransmission</type>
@@ -518,5 +518,5 @@
        <mechanicalReduction>1</mechanicalReduction>
      </actuator>
-   </transmission>
+  </transmission>
   <link name="l_hip_pitch_link">
     <collision>
@@ -539,5 +539,5 @@
     </inertial>
   </link>
-   <joint name="l_hip_roll" type="revolute">
+  <joint name="l_hip_roll" type="revolute">
     <parent link="l_hip_pitch_link"/>
     <child link="l_hip_roll_link"/>
@@ -546,6 +546,6 @@
     <limit velocity="6.5" effort="1000" lower="${-pi/2}" upper="${pi}" />
     <dynamics damping = "0.7"/>
-   </joint>
- <transmission name="l_hip_roll_tran">
+  </joint>
+  <transmission name="l_hip_roll_tran">
      <type>transmission_interface/SimpleTransmission</type>
      <joint name="l_hip_roll">
@@ -556,7 +556,7 @@
        <mechanicalReduction>1</mechanicalReduction>
      </actuator>
-   </transmission>
+  </transmission>
   <link name="l_hip_roll_link">
-     <collision>
+    <collision>
       <origin xyz="0 0 0" rpy="0 0 0"/>
       <geometry>
@@ -584,6 +584,6 @@
     <limit velocity="6.5" effort="1000" lower="${-pi/2}" upper="${pi/2}" />
     <dynamics damping = "0.7"/>
-   </joint>
- <transmission name="l_hip_yaw_tran">
+  </joint>
+  <transmission name="l_hip_yaw_tran">
      <type>transmission_interface/SimpleTransmission</type>
      <joint name="l_hip_yaw">
@@ -594,7 +594,7 @@
        <mechanicalReduction>1</mechanicalReduction>
      </actuator>
-   </transmission>
+  </transmission>
   <link name="l_hip_yaw_link">
-   <collision>
+    <collision>
       <origin xyz="0 0 0" rpy="0 0 0"/>
       <geometry>
@@ -622,6 +622,6 @@
     <limit velocity="6.5" effort="1000" lower="${-pi}" upper="${pi/2}" />
     <dynamics damping = "0.7"/>
-   </joint>
- <transmission name="l_knee_pitch_tran">
+  </joint>
+  <transmission name="l_knee_pitch_tran">
      <type>transmission_interface/SimpleTransmission</type>
      <joint name="l_knee_pitch">
@@ -632,5 +632,5 @@
        <mechanicalReduction>1</mechanicalReduction>
      </actuator>
-   </transmission>
+  </transmission>
   <link name="l_knee_pitch_link">
     <collision>
@@ -660,6 +660,6 @@
     <limit velocity="6.5" effort="1000" lower="${-pi/2}" upper="${pi}" />
     <dynamics damping = "0.7"/>
-   </joint>
- <transmission name="l_ankle_pitch_tran">
+  </joint>
+  <transmission name="l_ankle_pitch_tran">
      <type>transmission_interface/SimpleTransmission</type>
      <joint name="l_ankle_pitch">
@@ -670,5 +670,5 @@
        <mechanicalReduction>1</mechanicalReduction>
      </actuator>
-   </transmission>
+  </transmission>
   <link name="l_ankle_pitch_link">
     <collision>
@@ -698,6 +698,6 @@
     <limit velocity="6.5" effort="1000" lower="${-pi/2}" upper="${pi/2}" />
     <dynamics damping = "0.7"/>
-   </joint>
- <transmission name="l_ankle_roll_tran">
+  </joint>
+  <transmission name="l_ankle_roll_tran">
      <type>transmission_interface/SimpleTransmission</type>
      <joint name="l_ankle_roll">
@@ -708,5 +708,5 @@
        <mechanicalReduction>1</mechanicalReduction>
      </actuator>
-   </transmission>
+  </transmission>
   <link name="l_ankle_roll_link">
     <collision>
@@ -734,5 +734,5 @@
     <origin xyz="0 0 -0.135" rpy="0 0 0"/>
   </joint>
-<link name="l_foot_link">
+  <link name="l_foot_link">
     <collision>
       <origin xyz="0 0 -0.005" rpy="0 0 0"/>
@@ -754,6 +754,6 @@
     </inertial>
   </link>
-<!-- right leg -->
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